File: hardware/magnet_module/magnet/sensors.kicad_sch (KiCad schematic)
At the start: 0 parts

Commit message: sensor design
Parts:
- added J8: Conn_01x02_Pin, symbol Connector:Conn_01x02_Pin
- added R6: 10k, symbol Device:R
- added U6: 74LVC1G17, symbol 74xGxx:74LVC1G17
- added U7: SHT40-AD1B-R2, Leaf_Temperature:Sensirion_DFN-4_1.5x1.5mm_P0.8mm_SHT4x_NoCentralPad, symbol Leaf_Temperature:SHT4x
Connections:
- new net: J8.2 (Pin_2), R6.1, U6.2
- new net 3V3: J8.1 (Pin_1), U6.5 (VCC), U7.3 (VDD)
- new net GND: R6.2, U6.3 (GND), U7.4 (VSS)
- new net PRESSURE_OUT: U6.4
- new net TEMP.SCL: U7.2 (SCL)
- new net TEMP.SDA: U7.1 (SDA)
Other:
- note added: "To resistive pressure sensor (FSR400 series)"
