File: hardware/magnet_module/magnet/mcu.kicad_sch (KiCad schematic)
At the start: 1 part, among them U3 W25Q16JVSSIQ

Commit message: sensor design
Parts:
- added C10, C11, C12, C13, C14, C15, C16, C17, C18, C19: 0.1uF, symbol Device:C
- added D2: 150060YS75000, symbol Device:D
- added FB1, FB2: FerriteBead, symbol Device:FerriteBead
- added J9: STLINK-V3-MINIE, Leaf_Connectors:Tag-Connect_TC2070-IDC-NL_2x07_P1.27mm_Vertical, symbol Leaf_Connectors:STLINK-V3-MINIE-TagConnect
- added R10, R11, R7, R8, R9: 10k, symbol Device:R
- added R14: 220, symbol Device:R
- added SW1: SW_DIP_x02, symbol Switch:SW_DIP_x02
- added SW2, SW3: CK_PTS526_SK15_Switch, Leaf_Switch:CK_PTS526_SK15_Switch, symbol Leaf_Switch:CK_PTS526_SK15_Switch
- added U8: STM32G474RETx, Package_QFP:LQFP-64_10x10mm_P0.5mm, symbol MCU_ST_STM32G4:STM32G474RETx
- added U9: TXB0102RUT, Package_SO:TSSOP-8_3x3mm_P0.65mm, symbol Logic_LevelTranslator:TXB0102DCT
- added XTAL1: ASEMB-8.000MHZ-LC-T, Leaf_Clocks:ABRACON_ASE, symbol Leaf_Clocks:ASE-50.000MHZ-LC-T
Connections:
- net FLASH_~{CS}: now reaches U3.1 (~{CS})
- net FLASH_~{CS}: now also U8.34 (PB12)
- net FLASH_DO: now reaches U3.2 (DO(IO1))
- net FLASH_DO: now also U8.36 (PB14)
- net FLASH_~{WP}: now reaches U3.3 (IO2)
- net FLASH_~{WP}: now also R8.1
- net GND: now reaches U3.4 (GND)
- net GND: now also C10.2, C11.2, C12.2, C13.2, C14.2, C15.2, C16.2, C17.2, C18.2, C19.2, J9.11 (GNDDETECT), J9.5 (GND), J9.7 (GND), R14.2, SW1.3, SW1.4, SW2.1, SW2.2, SW3.1, SW3.2, U8.13 (PA1), U8.15 (VSS), U8.27 (VSSA), U8.31 (VSS), U8.47 (VSS), U8.63 (VSS), U9.2 (GND), XTAL1.2 (GND)
- net FLASH_DI: now reaches U3.5 (DI(IO0))
- net FLASH_DI: now also U8.37 (PB15)
- net FLASH_CLK: now reaches U3.6 (CLK)
- net FLASH_CLK: now also U8.35 (PB13)
- net FLASH_~{RST}: now reaches U3.7 (IO3)
- net FLASH_~{RST}: now also R7.1
- net 3V3: now reaches U3.8 (VCC)
- net 3V3: now also C11.1, C12.1, C14.1, C15.1, C16.1, C17.1, FB1.2, FB2.1, J9.3 (T_VCC), R10.1, R11.1, R7.2, R8.2, R9.1, U8.16 (VDD), U8.32 (VDD), U8.48 (VDD), U8.64 (VDD), U9.3 (VCCA), U9.6 (OE)
- new net: C10.1, FB2.2, XTAL1.4 (VDD)
- new net: D2.1 (K), R14.1
- new net 5V: C13.1, U9.7 (VCCB)
- new net 5V_SERVO0: U9.8 (B1)
- new net 5V_SERVO1: U9.1 (B2)
- new net BOOT: SW3.3 (K), SW3.4 (A), U8.61 (PB8)
- new net BUTTON0: U8.25 (PB1)
- new net BUTTON1: U8.26 (PB2)
- new net CANID0: R9.2, SW1.1, U8.10 (PC2)
- new net CANID1: R10.2, SW1.2, U8.11 (PC3)
- new net CANID2: R11.2, U8.12 (PA0)
- new net CELL.SCL: U8.38 (PC6)
- new net CELL.SDA: U8.39 (PC7)
- new net DEBUG_RX: J9.13 (T_VCP_RX), U8.8 (PC0)
- new net DEBUG_TX: J9.14 (T_VCP_TX), U8.9 (PC1)
- new net DM: U8.45 (PA11)
- new net DP: U8.46 (PA12)
- new net DRDY: U8.23 (PC5)
- new net GPIO0: U8.3 (PC14)
- new net GPIO1: U8.4 (PC15)
- new net OSC_IN: U8.5 (PF0), XTAL1.3 (OUTPUT)
- new net PRESSURE_IN: U8.24 (PB0)
- new net RX: U8.58 (PB5)
- new net SERVO0: U8.14 (PA2), U9.5 (A1)
- new net SERVO1: U8.17 (PA3), U9.4 (A2)
- new net SPARE0.SCL: U8.40 (PC8)
- new net SPARE0.SDA: U8.41 (PC9)
- new net SPARE1.SCL: U8.43 (PA9)
- new net SPARE1.SDA: U8.42 (PA8)
- new net STATUS_LED: D2.2 (A), U8.20 (PA6)
- new net STIM0: U8.52 (PC10)
- new net STIM1: U8.53 (PC11)
- new net STIM2: U8.54 (PC12)
- new net STIM3: U8.55 (PD2)
- new net SWCLK: J9.6 (T_SWCLK)
- new net SWIO: J9.4 (T_SWDIO)
- new net TEMP.SCL: U8.51 (PA15)
- new net TEMP.SDA: U8.50 (PA14)
- new net TX: U8.59 (PB6)
- new net VDDA: C18.1, FB1.1, U8.28 (VREF+), U8.29 (VDDA)
- new net ~{MCU_RST}: C19.1, J9.12 (T_NRST), SW2.3 (K), SW2.4 (A), U8.7 (PG10)
- no-connect marks 0 -> 8
Other:
- note added: "ADC1_IN12"
- note added: "CAN Addressing"
- note added: "Debug"
- note added: "Decoupling Capacitor Central"
- note added: "Device Type 0b00 = Pellet 0b01 = Magnet"
- note added: "External clock"
- note added: "FDCAN2_RX"
- note added: "FDCAN2_TX"
- note added: "I2C1_SCL"
- note added: "I2C1_SDA"
- note added: "I2C2_SCL"
- note added: "I2C2_SDA"
- note added: "I2C3_SCL"
- note added: "I2C3_SDA"
- note added: "I2C4_SCL"
- note added: "I2C4_SDA"
- note added: "If = 6mA"
- note added: "LPUART1_RX"
- note added: "LPUART1_TX"
- note added: "Module Address"
- note added: "Programming Flash"
- note added: "SPI2_MISO"
- note added: "SPI2_MOSI"
- note added: "SPI2_NSS"
- note added: "SPI2_SCK"
- note added: "Servo Level Shifting"
- note added: "Status LED"
- note added: "TIM2_CH3"
- note added: "TIM5_CH4"
- note added: "USB_DM"
- note added: "USB_DN"
- note added: "Vf = 2V"
- moved on the sheet: U3

Commit message: fix erc errors
Connections:
- net GND: no longer J9.11 (GNDDETECT)
- net SWCLK: now also U8.50 (PA14)
- net SWIO: now also U8.49 (PA13)
- net TEMP.SDA: now also U8.62 (PB9); no longer U8.50 (PA14)
- no-connect marks 8 -> 18
Other:
- note added: "SWCLK-JTCK"
- note added: "SWDIO-JTMS"
Changed lines of the file:
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@@
 	)
 	(junction
-		(at 26.67 85.09)
-		(diameter 0)
-		(color 0 0 0 0)
-	)
-	(junction
 		(at 161.29 29.21)
 		(diameter 0)
@@
 	)
 	(no_connect
+		(at 171.45 53.34)
+	)
+	(no_connect
+		(at 171.45 104.14)
+	)
+	(no_connect
+		(at 27.94 82.55)
+	)
+	(no_connect
+		(at 171.45 111.76)
+	)
+	(no_connect
 		(at 135.89 76.2)
 	)
@@
 	)
 	(no_connect
+		(at 171.45 60.96)
+	)
+	(no_connect
 		(at 58.42 80.01)
 	)
@@
 		(at 58.42 72.39)
 	)
+	(no_connect
+		(at 171.45 68.58)
+	)
+	(no_connect
+		(at 171.45 114.3)
+	)
+	(no_connect
+		(at 171.45 96.52)
+	)
+	(no_connect
+		(at 171.45 93.98)
+	)
+	(no_connect
+		(at 171.45 55.88)
+	)
 	(bus_entry
 		(at 189.23 101.6)
@@
 	)
 	(bus_entry
-		(at 194.31 81.28)
-		(size -2.54 -2.54)
-		(stroke
-			(width 0)
-			(type default)
-		)
-	)
-	(bus_entry
 		(at 111.76 81.28)
 		(size 2.54 2.54)
@@
 		)
 	)
-	(bus
-		(pts
-			(xy 194.31 81.28) (xy 194.31 83.82)
-		)
-		(stroke
-			(width 0)
-			(type default)
-		)
-	)
 	(wire
 		(pts
@@
 		)
 	)
-	(bus
-		(pts
-			(xy 194.31 81.28) (xy 194.31 80.01)
-		)
-		(stroke
-			(width 0)
-			(type default)
-		)
-	)
 	(wire
 		(pts
@@
 	(wire
 		(pts
-			(xy 26.67 82.55) (xy 26.67 85.09)
-		)
-		(stroke
-			(width 0)
-			(type default)
-		)
-	)
-	(wire
-		(pts
 			(xy 193.04 66.04) (xy 171.45 66.04)
 		)
@@
 	(wire
 		(pts
-			(xy 26.67 82.55) (xy 27.94 82.55)
-		)
-		(stroke
-			(width 0)
-			(type default)
-		)
-	)
-	(wire
-		(pts
 			(xy 156.21 132.08) (xy 156.21 133.35)
 		)
@@
 		)
 	)
-	(wire
+	(bus
 		(pts
-			(xy 140.97 177.8) (xy 144.78 177.8)
+			(xy 194.31 83.82) (xy 195.58 83.82)
 		)
 		(stroke
@@
 	(wire
 		(pts
-			(xy 156.21 38.1) (xy 156.21 36.83)
+			(xy 140.97 177.8) (xy 144.78 177.8)
 		)
 		(stroke
@@
 	(wire
 		(pts
-			(xy 245.11 149.86) (xy 217.17 149.86)
+			(xy 156.21 38.1) (xy 156.21 36.83)
 		)
 		(stroke
@@
 	(wire
 		(pts
-			(xy 20.32 110.49) (xy 20.32 111.76)
+			(xy 245.11 149.86) (xy 217.17 149.86)
 		)
 		(stroke
@@
 	(wire
 		(pts
-			(xy 57.15 111.76) (xy 57.15 113.03)
+			(xy 20.32 110.49) (xy 20.32 111.76)
 		)
 		(stroke
@@
 	(wire
 		(pts
-			(xy 171.45 78.74) (xy 191.77 78.74)
+			(xy 57.15 111.76) (xy 57.15 113.03)
 		)
 		(stroke
@@
 		)
 	)
+	(text "SWCLK-JTCK"
+		(exclude_from_sim no)
+		(at 179.07 78.74 0)
+		(effects
+			(font
+				(size 1.27 1.27)
+			)
+			(justify left bottom)
+		)
+	)
 	(text "LPUART1_RX"
 		(exclude_from_sim no)
@@
 	(text "I2C1_SDA"
 		(exclude_from_sim no)
-		(at 186.69 77.47 0)
+		(at 187.198 108.204 0)
 		(effects
 			(font
@@
 	(text "I2C1_SCL"
 		(exclude_from_sim no)
-		(at 186.69 80.01 0)
+		(at 186.182 80.518 0)
 		(effects
 			(font
@@
 		)
 	)
+	(text "SWDIO-JTMS"
+		(exclude_from_sim no)
+		(at 185.166 75.692 0)
+		(effects
+			(font
+				(size 1.27 1.27)
+			)
+		)
+	)
 	(label "BOOT"
 		(at 69.85 109.22 0)
@@
 		)
 	)
+	(label "SWIO"
+		(at 171.45 76.2 0)
+		(fields_autoplaced yes)
+		(effects
+			(font
+				(size 1.27 1.27)
+			)
+			(justify left bottom)
+		)
+	)
 	(label "CANID3"
 		(at 132.08 189.23 180)
@@
 	)
 	(label "TEMP.SDA"
-		(at 171.45 78.74 0)
+		(at 171.45 109.22 0)
 		(fields_autoplaced yes)
 		(effects
@@
 		)
 	)
+	(label "SWCLK"
+		(at 171.45 78.74 0)
+		(fields_autoplaced yes)
+		(effects
+			(font
+				(size 1.27 1.27)
+			)
+			(justify left bottom)
+		)
+	)
 	(label "3V3"
 		(at 180.34 29.21 180)
@@
 	(hierarchical_label "TEMP{I2C}"
 		(shape bidirectional)
-		(at 194.31 80.01 0)
+		(at 195.58 83.82 0)
 		(fields_autoplaced yes)
 		(effects
@@
 		(pin "1"
 		)
-		(instances
-			(project ""
-				(path "/aa5044b8-67cd-4b5a-a593-0df9431eb095/286cc8bf-34fd-48cd-9d6c-58653d0694aa"
-					(reference "U3")
-					(unit 1)
-				)
-			)
-		)
 	)
 	(symbol
@@
 		(pin "45"
 		)
-		(instances
-			(project ""
-				(path "/aa5044b8-67cd-4b5a-a593-0df9431eb095/286cc8bf-34fd-48cd-9d6c-58653d0694aa"
-					(reference "U8")
-					(unit 1)
-				)
-			)
-		)
 	)
