File: hardware/jetson_breakout/jetson_breakout.kicad_sch (KiCad schematic)
At the start: 0 parts

Commit message: Releases layout for pellet, magnet, and Jetson breakout boards.
Parts:
- added U3: Leaf_Logo, Leaf_Mechanical:leaf_logo_small, symbol Leaf_Graphics:Leaf_Logo
Changed lines of the file:
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@@
 	(title_block
 		(title "Jetson AGX Orin CAN Adapter")
-		(date "2024-07-16")
+		(date "2024-07-26")
 		(rev "v1.0")
 		(company "Christie Lab, CU Anschutz")
@@
 		)
 	)
+	(symbol
+		(lib_id "Leaf_Graphics:Leaf_Logo")
+		(at 31.75 177.8 0)
+		(unit 1)
+		(exclude_from_sim no)
+		(in_bom no)
+		(on_board yes)
+		(dnp no)
+		(fields_autoplaced yes)
+		(property "Reference" "U3"
+			(at 33.02 176.5299 0)
+			(effects
+				(font
+					(size 1.27 1.27)
+				)
+				(justify left)
+			)
+		)
+		(property "Value" "Leaf_Logo"
+			(at 33.02 179.0699 0)
+			(effects
+				(font
+					(size 1.27 1.27)
+				)
+				(justify left)
+			)
+		)
+		(property "Footprint" "Leaf_Mechanical:leaf_logo_small"
+			(at 31.75 177.8 0)
+			(effects
+				(font
+					(size 1.27 1.27)
+				)
+				(hide yes)
+			)
+		)
+		(property "Datasheet" ""
+			(at 31.75 177.8 0)
+			(effects
+				(font
+					(size 1.27 1.27)
+				)
+				(hide yes)
+			)
+		)
+		(property "Description" ""
+			(at 31.75 177.8 0)
+			(effects
+				(font
+					(size 1.27 1.27)
+				)
+				(hide yes)
+			)
+		)
+		(instances
+			(project ""
+				(path "/2f8e404a-f8f0-4824-bb86-c9c070099b28"
+					(reference "U3")
+					(unit 1)
+				)
+			)
+		)
+	)
