File: hardware/jetson_breakout/orin.kicad_sch (KiCad schematic)
At the start: 1 part, among them J1 Jetson AGX Orin 40pin Header

Commit message: Releases layout for pellet, magnet, and Jetson breakout boards.
Parts:
- J1: footprint Connector_PinHeader_2.54mm:PinHeader_2x20_P2.54mm_Vertical -> Connector_PinSocket_2.54mm:PinSocket_2x20_P2.54mm_Vertical; LCSC (none) -> C2977589; MPN SSW-120-01-T-D-LL -> 2.54-2*20
Other:
- note added: "All signals at logic level 3.3V"
- note removed: "Orin: input = out of header, output = into header"
- company: (none) -> Christie Lab, CU Anschutz
- title: (none) -> Jetson AGX Orin CAN Adapter - Jetson
Changed lines of the file:
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@@
 	(generator_version "8.0")
 	(paper "A4")
+	(title_block
+		(title "Jetson AGX Orin CAN Adapter - Jetson")
+		(date "2024-07-26")
+		(rev "v1.0")
+		(company "Christie Lab, CU Anschutz")
+		(comment 1 "Prepared by LeafLabs, LLC")
+	)
 	(junction
 		(at 133.35 132.08)
@@
 	(junction
 		(at 143.51 132.08)
+		(diameter 0)
+		(color 0 0 0 0)
+	)
+	(junction
+		(at 128.27 135.89)
 		(diameter 0)
 		(color 0 0 0 0)
@@
 	(wire
 		(pts
-			(xy 128.27 132.08) (xy 128.27 133.35)
+			(xy 128.27 132.08) (xy 128.27 135.89)
 		)
 		(stroke
@@
 	(wire
 		(pts
+			(xy 128.27 135.89) (xy 128.27 138.43)
+		)
+		(stroke
+			(width 0)
+			(type default)
+		)
+	)
+	(wire
+		(pts
 			(xy 143.51 132.08) (xy 146.05 132.08)
 		)
@@
 		)
 	)
-	(text "Orin: \ninput = out of header, \noutput = into header"
+	(text "All signals at logic level 3.3V"
 		(exclude_from_sim no)
-		(at 172.974 90.424 0)
+		(at 177.292 72.898 0)
 		(effects
 			(font
@@
 				)
 				(justify left)
+			)
+		)
+	)
+	(symbol
+		(lib_id "power:PWR_FLAG")
+		(at 128.27 135.89 90)
+		(unit 1)
+		(exclude_from_sim no)
+		(in_bom yes)
+		(on_board yes)
+		(dnp no)
+		(fields_autoplaced yes)
+		(property "Reference" "#FLG01"
+			(at 126.365 135.89 0)
+			(effects
+				(font
+					(size 1.27 1.27)
+				)
+				(hide yes)
+			)
+		)
+		(property "Value" "PWR_FLAG"
+			(at 124.46 135.8899 90)
+			(effects
+				(font
+					(size 1.27 1.27)
+				)
+				(justify left)
+			)
+		)
+		(property "Footprint" ""
+			(at 128.27 135.89 0)
+			(effects
+				(font
+					(size 1.27 1.27)
+				)
+				(hide yes)
+			)
+		)
+		(property "Datasheet" "~"
+			(at 128.27 135.89 0)
+			(effects
+				(font
+					(size 1.27 1.27)
+				)
+				(hide yes)
+			)
+		)
+		(property "Description" "Special symbol for telling ERC where power comes from"
+			(at 128.27 135.89 0)
+			(effects
+				(font
+					(size 1.27 1.27)
+				)
+				(hide yes)
+			)
+		)
+		(pin "1"
+		)
+		(instances
+			(project ""
+				(path "/2f8e404a-f8f0-4824-bb86-c9c070099b28/f93aa4ed-249c-403a-91f0-1440dbc911e5"
+					(reference "#FLG01")
+					(unit 1)
+				)
 			)
 		)
@@
 			)
 		)
-		(property "Footprint" "Connector_PinHeader_2.54mm:PinHeader_2x20_P2.54mm_Vertical"
+		(property "Footprint" "Connector_PinSocket_2.54mm:PinSocket_2x20_P2.54mm_Vertical"
 			(at 137.16 64.77 0)
 			(effects
@@
 			)
 		)
-		(property "Datasheet" ""
+		(property "Datasheet" "https://jetsonhacks.com/nvidia-jetson-agx-orin-gpio-header-pinout/"
 			(at 137.16 64.77 0)
 			(effects
@@
 			)
 		)
-		(property "MPN" "SSW-120-01-T-D-LL"
+		(property "MPN" "2.54-2*20"
 			(at 137.16 64.77 0)
 			(effects
@@
 		)
 		(property "Sim.Pins" ""
+			(at 137.16 64.77 0)
+			(effects
+				(font
+					(size 1.27 1.27)
+				)
+				(hide yes)
+			)
+		)
+		(property "LCSC" "C2977589"
 			(at 137.16 64.77 0)
 			(effects
@@
 	(symbol
 		(lib_id "power:GND")
-		(at 128.27 133.35 0)
+		(at 128.27 138.43 0)
 		(unit 1)
 		(exclude_from_sim no)
@@
 		(fields_autoplaced yes)
 		(property "Reference" "#PWR01"
-			(at 128.27 139.7 0)
+			(at 128.27 144.78 0)
 			(effects
 				(font
@@
 		)
 		(property "Value" "GND"
+			(at 128.27 143.51 0)
+			(effects
+				(font
+					(size 1.27 1.27)
+				)
+			)
+		)
+		(property "Footprint" ""
 			(at 128.27 138.43 0)
 			(effects
@@
 					(size 1.27 1.27)
 				)
-			)
-		)
-		(property "Footprint" ""
-			(at 128.27 133.35 0)
-			(effects
-				(font
-					(size 1.27 1.27)
-				)
 				(hide yes)
 			)
 		)
 		(property "Datasheet" ""
-			(at 128.27 133.35 0)
+			(at 128.27 138.43 0)
 			(effects
 				(font
@@
 		)
 		(property "Description" "Power symbol creates a global label with name \"GND\" , ground"
-			(at 128.27 133.35 0)
-			(effects
-				(font
+			(at 128.27 138.43 0)
+			(effects
+				(font
