File: hardware/jetson_breakout/power.kicad_sch (KiCad schematic)
At the start: 3 parts, among them J4 Barrel_Jack_Switch

Commit message: Releases layout for pellet, magnet, and Jetson breakout boards.
Parts:
- D2: LCSC (none) -> C5252984
- J4: LCSC (none) -> C5280493
- R2: LCSC (none) -> C4190; MPN RC0603FR-072K2L -> 0603WAF2201T5E
Other:
- company: (none) -> Christie Lab, CU Anschutz
- title: (none) -> Jetson AGX Orin CAN Adapter - Power
Changed lines of the file:
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@@
 	(generator_version "8.0")
 	(paper "A4")
+	(title_block
+		(title "Jetson AGX Orin CAN Adapter - Power")
+		(date "2024-07-26")
+		(rev "v1.0")
+		(company "Christie Lab, CU Anschutz")
+		(comment 1 "Prepared by LeafLabs, LLC")
+	)
 	(junction
 		(at 135.89 96.52)
@@
 		(pts
 			(xy 137.16 96.52) (xy 135.89 96.52)
+		)
+		(stroke
+			(width 0)
+			(type default)
+		)
+	)
+	(wire
+		(pts
+			(xy 153.67 116.84) (xy 153.67 113.03)
 		)
 		(stroke
@@
 			)
 		)
+		(property "LCSC" "C5280493"
+			(at 119.38 93.98 0)
+			(effects
+				(font
+					(size 1.27 1.27)
+				)
+				(hide yes)
+			)
+		)
 		(pin "3"
 		)
@@
 	(symbol
 		(lib_id "power:GND")
-		(at 153.67 113.03 0)
+		(at 153.67 116.84 0)
 		(unit 1)
 		(exclude_from_sim no)
@@
 		(fields_autoplaced yes)
 		(property "Reference" "#PWR08"
-			(at 153.67 119.38 0)
+			(at 153.67 123.19 0)
 			(effects
 				(font
@@
 		)
 		(property "Value" "GND"
-			(at 153.67 118.11 0)
+			(at 153.67 121.92 0)
 			(effects
 				(font
@@
 		)
 		(property "Footprint" ""
-			(at 153.67 113.03 0)
+			(at 153.67 116.84 0)
 			(effects
 				(font
@@
 		)
 		(property "Datasheet" ""
-			(at 153.67 113.03 0)
+			(at 153.67 116.84 0)
 			(effects
 				(font
@@
 		)
 		(property "Description" "Power symbol creates a global label with name \"GND\" , ground"
-			(at 153.67 113.03 0)
+			(at 153.67 116.84 0)
 			(effects
 				(font
@@
 			)
 		)
+		(property "LCSC" "C5252984"
+			(at 153.67 96.52 0)
+			(effects
+				(font
+					(size 1.27 1.27)
+				)
+				(hide yes)
+			)
+		)
 		(pin "1"
 		)
@@
 			)
 		)
-		(property "MPN" "RC0603FR-072K2L"
+		(property "MPN" "0603WAF2201T5E"
 			(at 153.67 109.22 0)
 			(effects
@@
 			(at 153.67 109.22 0)
 			(effects
+				(font
+					(size 1.27 1.27)
+				)
+				(hide yes)
+			)
+		)
+		(property "LCSC" "C4190"
+			(at 153.67 109.22 0)
+			(effects
