File: hardware/magnet_module/servo.kicad_sch (KiCad schematic)
At the start: 5 parts, among them J21 Conn_01x03_Pin, J4 Conn_01x03_Pin, U6 TXB0102RUT

Commit message: Releases layout for pellet, magnet, and Jetson breakout boards.
Parts:
- C12, C13: LCSC (none) -> C14663; MPN CC0603KRX7R7BB104 -> CC0603KRX7R9BB104
- J21, J4: LCSC (none) -> C144394
- U6: value TXB0102RUT -> TXB0102DCU; footprint Package_SO:TSSOP-8_3x3mm_P0.65mm -> Package_SO:VSSOP-8_2.3x2mm_P0.5mm; LCSC (none) -> C60709; MPN TXB0102RUT -> TXB0102DCUR
Connections:
- net 5V_SERVO0: now also U6.1 (B2); no longer U6.8 (B1)
- net 5V_SERVO1: now also U6.8 (B1); no longer U6.1 (B2)
- net SERVO0: now also U6.4 (A2); no longer U6.5 (A1)
- net SERVO1: now also U6.5 (A1); no longer U6.4 (A2)
Changed lines of the file:
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@@
 	(title_block
 		(title "Autotrainer Magnet Module - Servos")
-		(date "2024-07-09")
+		(date "2024-07-26")
 		(rev "v1.0")
 		(company "Christie Lab, CU-Anschutz")
@@
 	)
 	(label "5V_SERVO0"
-		(at 76.2 109.22 0)
+		(at 76.2 114.3 0)
 		(fields_autoplaced yes)
 		(effects
@@
 	)
 	(label "SERVO1"
-		(at 55.88 114.3 180)
+		(at 55.88 109.22 180)
 		(fields_autoplaced yes)
 		(effects
@@
 	)
 	(label "SERVO0"
-		(at 55.88 109.22 180)
+		(at 55.88 114.3 180)
 		(fields_autoplaced yes)
 		(effects
@@
 	)
 	(label "5V_SERVO1"
-		(at 76.2 114.3 0)
+		(at 76.2 109.22 0)
 		(fields_autoplaced yes)
 		(effects
@@
 			)
 		)
-		(property "MPN" "CC0603KRX7R7BB104"
+		(property "MPN" "CC0603KRX7R9BB104"
+			(at 72.39 97.79 0)
+			(effects
+				(font
+					(size 1.27 1.27)
+				)
+				(hide yes)
+			)
+		)
+		(property "LCSC" "C14663"
 			(at 72.39 97.79 0)
 			(effects
@@
 		(on_board yes)
 		(dnp no)
-		(fields_autoplaced yes)
 		(property "Reference" "U6"
-			(at 68.2341 124.46 0)
+			(at 74.676 124.46 0)
 			(effects
 				(font
@@
 			)
 		)
-		(property "Value" "TXB0102RUT"
-			(at 68.2341 127 0)
-			(effects
-				(font
-					(size 1.27 1.27)
-				)
-				(justify left)
-			)
-		)
-		(property "Footprint" "Package_SO:TSSOP-8_3x3mm_P0.65mm"
+		(property "Value" "TXB0102DCU"
+			(at 74.676 127 0)
+			(effects
+				(font
+					(size 1.27 1.27)
+				)
+			)
+		)
+		(property "Footprint" "Package_SO:VSSOP-8_2.3x2mm_P0.5mm"
 			(at 66.04 125.73 0)
 			(effects
@@
 			)
 		)
-		(property "MPN" "TXB0102RUT"
+		(property "MPN" "TXB0102DCUR"
+			(at 66.04 111.76 0)
+			(effects
+				(font
+					(size 1.27 1.27)
+				)
+				(hide yes)
+			)
+		)
+		(property "LCSC" "C60709"
 			(at 66.04 111.76 0)
 			(effects
@@
 			)
 		)
+		(property "LCSC" "C144394"
+			(at 133.35 99.06 0)
+			(effects
+				(font
+					(size 1.27 1.27)
+				)
+				(hide yes)
+			)
+		)
 		(pin "2"
 		)
@@
 		)
 		(property "MPN" "B3B-XH-A"
+			(at 133.35 124.46 0)
+			(effects
+				(font
+					(size 1.27 1.27)
+				)
+				(hide yes)
+			)
+		)
+		(property "LCSC" "C144394"
 			(at 133.35 124.46 0)
 			(effects
@@
 			)
 		)
-		(property "MPN" "CC0603KRX7R7BB104"
+		(property "MPN" "CC0603KRX7R9BB104"
 			(at 59.69 97.79 0)
 			(effects
+				(font
+					(size 1.27 1.27)
+				)
+				(hide yes)
+			)
+		)
+		(property "LCSC" "C14663"
+			(at 59.69 97.79 0)
+			(effects
