File: hardware/magnet_module/mcu.kicad_sch (KiCad schematic)
At the start: 36 parts, among them J9 STLINK-V3-MINIE, SW1 SW_DIP_x02, SW2 CK_PTS526_SK15_Switch, SW3 CK_PTS526_SK15_Switch, U15 W25Q16JVSSIQ, U8 STM32G474RETx

Commit message: Update Magnet BOM for part availability
Parts:
- D2: LCSC C9900012286 -> C6784997
Changed lines of the file:
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@@
 			)
 		)
-		(property "LCSC" "C9900012286"
+		(property "LCSC" "C6784997"
 			(at 40.64 26.67 0)
 			(effects
