File: hardware/pellet_module/stim.kicad_sch (KiCad schematic)
At the start: 16 parts, among them J11 Conn_Coaxial, J12 Conn_01x03_Pin, J13 Conn_01x03_Pin, J14 Conn_01x03_Pin, J15 Conn_Coaxial, J16 Conn_Coaxial, J17 Conn_Coaxial, J18 Conn_Coaxial, U7 TXB0104RUT

Commit message: add test points, mpns, datasheets
Parts:
- C32, C33, C34: footprint (none) -> Capacitor_SMD:C_0603_1608Metric; MPN (none) -> CC0603ZRY5V9BB104
- J11, J15, J16, J17, J18: MPN (none) -> CONMHF1-SMD-T
- J12, J13, J14: MPN (none) -> 61300311121
- R14, R15, R16, R22: MPN (none) -> RC0603FR-0710KL
- U7: MPN (none) -> TXB0104RUT
Changed lines of the file:
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@@
+			)
+		)
+		(property "MPN" "CONMHF1-SMD-T"
+			(at 48.26 34.29 0)
+			(effects
+				(font
+					(size 1.27 1.27)
+				)
+				(hide yes)
 			)
 		)
@@
 			)
 		)
-		(property "MPN" ""
+		(property "MPN" "RC0603FR-0710KL"
 			(at 50.8 116.84 0)
 			(effects
@@
 			)
 		)
-		(property "MPN" ""
+		(property "MPN" "RC0603FR-0710KL"
 			(at 50.8 86.36 0)
 			(effects
@@
 			)
 		)
-		(property "MPN" ""
+		(property "MPN" "RC0603FR-0710KL"
 			(at 50.8 101.6 0)
 			(effects
@@
 			)
 		)
-		(property "MPN" ""
+		(property "MPN" "RC0603FR-0710KL"
 			(at 35.56 30.48 0)
 			(effects
@@
 			)
 		)
-		(property "Footprint" ""
+		(property "Footprint" "Capacitor_SMD:C_0603_1608Metric"
 			(at 38.4048 41.91 0)
 			(effects
@@
 			)
 		)
-		(property "MPN" ""
+		(property "MPN" "CC0603ZRY5V9BB104"
 			(at 39.37 38.1 0)
 			(effects
@@
 		)
 		(property "Description" "4-Bit Bidirectional Voltage-Level Translator, Auto Direction Sensing and ±15-kV ESD Protection, 1.2 - 3.6V APort, 1.65 - 5.5V BPort, Texas_PUQFN-12"
+			(at 172.72 96.52 0)
+			(effects
+				(font
+					(size 1.27 1.27)
+				)
+				(hide yes)
+			)
+		)
+		(property "MPN" "TXB0104RUT"
 			(at 172.72 96.52 0)
 			(effects
@@
 			)
 		)
+		(property "MPN" "61300311121"
+			(at 59.69 104.14 0)
+			(effects
+				(font
+					(size 1.27 1.27)
+				)
+				(hide yes)
+			)
+		)
 		(pin "2"
 		)
@@
 			)
 		)
+		(property "MPN" "CONMHF1-SMD-T"
+			(at 220.98 87.63 0)
+			(effects
+				(font
+					(size 1.27 1.27)
+				)
+				(hide yes)
+			)
+		)
 		(pin "1"
 		)
@@
 		)
 		(property "Description" "coaxial connector (BNC, SMA, SMB, SMC, Cinch/RCA, LEMO, ...)"
+			(at 220.98 102.87 0)
+			(effects
+				(font
+					(size 1.27 1.27)
+				)
+				(hide yes)
+			)
+		)
+		(property "MPN" "CONMHF1-SMD-T"
 			(at 220.98 102.87 0)
 			(effects
@@
 			)
 		)
+		(property "MPN" "61300311121"
+			(at 59.69 119.38 0)
+			(effects
+				(font
+					(size 1.27 1.27)
+				)
+				(hide yes)
+			)
+		)
 		(pin "2"
 		)
@@
 			)
 		)
+		(property "MPN" "CONMHF1-SMD-T"
+			(at 220.98 71.12 0)
+			(effects
+				(font
+					(size 1.27 1.27)
+				)
+				(hide yes)
+			)
+		)
 		(pin "1"
 		)
@@
 			)
 		)
-		(property "Footprint" ""
+		(property "Footprint" "Capacitor_SMD:C_0603_1608Metric"
 			(at 182.88 75.2348 0)
 			(effects
@@
 			)
 		)
-		(property "MPN" ""
+		(property "MPN" "CC0603ZRY5V9BB104"
 			(at 179.07 76.2 0)
 			(effects
@@
 			)
 		)
+		(property "MPN" "61300311121"
+			(at 59.69 88.9 0)
+			(effects
+				(font
+					(size 1.27 1.27)
+				)
+				(hide yes)
+			)
+		)
 		(pin "2"
 		)
@@
 		)
 		(property "Description" "coaxial connector (BNC, SMA, SMB, SMC, Cinch/RCA, LEMO, ...)"
+			(at 220.98 121.92 0)
+			(effects
+				(font
+					(size 1.27 1.27)
+				)
+				(hide yes)
+			)
+		)
+		(property "MPN" "CONMHF1-SMD-T"
 			(at 220.98 121.92 0)
 			(effects
@@
 			)
 		)
-		(property "Footprint" ""
+		(property "Footprint" "Capacitor_SMD:C_0603_1608Metric"
 			(at 162.56 75.2348 0)
 			(effects
@@
 			)
 		)
-		(property "MPN" ""
+		(property "MPN" "CC0603ZRY5V9BB104"
 			(at 166.37 76.2 0)
 			(effects

Commit message: add titles, ESD protection, make changes requested by Ryan
Parts:
- removed J12, J13, J14: Conn_01x03_Pin, symbol Connector:Conn_01x03_Pin
- added J12, J13, J14: Conn_01x02_Pin, symbol Connector:Conn_01x02_Pin
- added J21: Conn_Coaxial, symbol Connector:Conn_Coaxial
Connections:
- net GND: now also J21.2 (Ext)
- net LIMIT0: now also J12.2 (Pin_2)
- net LIMIT1: now also J13.2 (Pin_2)
- net LIMIT2: now also J14.2 (Pin_2)
- net at R16.1: now also J14.1 (Pin_1)
- net at R14.1: now also J12.1 (Pin_1)
- net at R15.1: now also J13.1 (Pin_1)
- new net STATUS_OUT: J21.1 (In)
- no-connect marks 3 -> 0
Other:
- note added: "Analog status indicator"
- note removed: "NO"
- company: (none) -> Christie Lab, CU-Anschutz
- title: (none) -> Autotrainer Pellet Module - External IO

Commit message: update connectors to right angle / update to bnc connector
Parts:
- J11, J15, J16, J17, J18, J21: MPN CONMHF1-SMD-T -> CONBNC002
Changed lines of the file:
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@@
 			)
 		)
-		(property "MPN" "CONMHF1-SMD-T"
+		(property "MPN" "CONBNC002"
 			(at 48.26 34.29 0)
 			(effects
@@
 			)
 		)
-		(property "MPN" "CONMHF1-SMD-T"
+		(property "MPN" "CONBNC002"
 			(at 49.53 153.67 0)
 			(effects
@@
 			)
 		)
-		(property "MPN" "CONMHF1-SMD-T"
+		(property "MPN" "CONBNC002"
 			(at 220.98 87.63 0)
 			(effects
@@
 			)
 		)
-		(property "MPN" "CONMHF1-SMD-T"
+		(property "MPN" "CONBNC002"
 			(at 220.98 102.87 0)
 			(effects
@@
 			)
 		)
-		(property "MPN" "CONMHF1-SMD-T"
+		(property "MPN" "CONBNC002"
 			(at 220.98 71.12 0)
 			(effects
@@
 			)
 		)
-		(property "MPN" "CONMHF1-SMD-T"
+		(property "MPN" "CONBNC002"
 			(at 220.98 121.92 0)
 			(effects

Commit message: * Add footprints for every part * Change power LED from 20mA to 4mA * Edit symbols to match footprints (EPAD -> pin numbers) to eliminate errors on import to pcbnew
Parts:
- J11, J15, J16, J17, J18, J21: footprint (none) -> Leaf_Connectors:CONBNC002
- J12, J13, J14: footprint (none) -> Connector_PinHeader_2.54mm:PinHeader_1x02_P2.54mm_Vertical; MPN (none) -> 61300211121
- R14, R15, R16, R22: footprint (none) -> Resistor_SMD:R_0603_1608Metric
Changed lines of the file:
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@@
 			)
 		)
-		(property "Footprint" ""
+		(property "Footprint" "Leaf_Connectors:CONBNC002"
 			(at 48.26 34.29 0)
 			(effects
@@
 			)
 		)
-		(property "Footprint" ""
+		(property "Footprint" "Leaf_Connectors:CONBNC002"
 			(at 49.53 153.67 0)
 			(effects
@@
 			)
 		)
-		(property "Footprint" ""
+		(property "Footprint" "Resistor_SMD:R_0603_1608Metric"
 			(at 50.8 118.618 90)
 			(effects
@@
 			)
 		)
-		(property "Footprint" ""
+		(property "Footprint" "Resistor_SMD:R_0603_1608Metric"
 			(at 50.8 88.138 90)
 			(effects
@@
 			)
 		)
-		(property "Footprint" ""
+		(property "Footprint" "Resistor_SMD:R_0603_1608Metric"
 			(at 50.8 103.378 90)
 			(effects
@@
 			)
 		)
-		(property "Footprint" ""
+		(property "Footprint" "Resistor_SMD:R_0603_1608Metric"
 			(at 33.782 30.48 90)
 			(effects
@@
 			)
 		)
-		(property "Footprint" ""
+		(property "Footprint" "Connector_PinHeader_2.54mm:PinHeader_1x02_P2.54mm_Vertical"
 			(at 59.69 101.6 0)
 			(effects
@@
 		)
 		(property "Description" "Generic connector, single row, 01x02, script generated"
+			(at 59.69 101.6 0)
+			(effects
+				(font
+					(size 1.27 1.27)
+				)
+				(hide yes)
+			)
+		)
+		(property "MPN" "61300211121"
 			(at 59.69 101.6 0)
 			(effects
@@
 			)
 		)
-		(property "Footprint" ""
+		(property "Footprint" "Connector_PinHeader_2.54mm:PinHeader_1x02_P2.54mm_Vertical"
 			(at 59.69 86.36 0)
 			(effects
@@
 			)
 		)
+		(property "MPN" "61300211121"
+			(at 59.69 86.36 0)
+			(effects
+				(font
+					(size 1.27 1.27)
+				)
+				(hide yes)
+			)
+		)
 		(pin "2"
 		)
@@
 			)
 		)
-		(property "Footprint" ""
+		(property "Footprint" "Leaf_Connectors:CONBNC002"
 			(at 220.98 87.63 0)
 			(effects
@@
 			)
 		)
-		(property "Footprint" ""
+		(property "Footprint" "Leaf_Connectors:CONBNC002"
 			(at 220.98 102.87 0)
 			(effects
@@
 			)
 		)
-		(property "Footprint" ""
+		(property "Footprint" "Connector_PinHeader_2.54mm:PinHeader_1x02_P2.54mm_Vertical"
 			(at 59.69 116.84 0)
 			(effects
@@
 		)
 		(property "Description" "Generic connector, single row, 01x02, script generated"
+			(at 59.69 116.84 0)
+			(effects
+				(font
+					(size 1.27 1.27)
+				)
+				(hide yes)
+			)
+		)
+		(property "MPN" "61300211121"
 			(at 59.69 116.84 0)
 			(effects
@@
 			)
 		)
-		(property "Footprint" ""
+		(property "Footprint" "Leaf_Connectors:CONBNC002"
 			(at 220.98 71.12 0)
 			(effects
@@
 			)
 		)
-		(property "Footprint" ""
+		(property "Footprint" "Leaf_Connectors:CONBNC002"
 			(at 220.98 121.92 0)
 			(effects

Commit message: update mechanicals based on dan's comments
Parts:
- J12, J13, J14: footprint Connector_PinHeader_2.54mm:PinHeader_1x02_P2.54mm_Vertical -> Connector_PinHeader_2.54mm:PinHeader_1x02_P2.54mm_Horizontal; MPN 61300211121 -> M20-9750242
Changed lines of the file:
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@@
 			)
 		)
-		(property "Footprint" "Connector_PinHeader_2.54mm:PinHeader_1x02_P2.54mm_Vertical"
+		(property "Footprint" "Connector_PinHeader_2.54mm:PinHeader_1x02_P2.54mm_Horizontal"
 			(at 59.69 101.6 0)
 			(effects
@@
 			)
 		)
-		(property "MPN" "61300211121"
+		(property "MPN" "M20-9750242"
 			(at 59.69 101.6 0)
 			(effects
@@
 			)
 		)
-		(property "Footprint" "Connector_PinHeader_2.54mm:PinHeader_1x02_P2.54mm_Vertical"
+		(property "Footprint" "Connector_PinHeader_2.54mm:PinHeader_1x02_P2.54mm_Horizontal"
 			(at 59.69 86.36 0)
 			(effects
@@
 			)
 		)
-		(property "MPN" "61300211121"
+		(property "MPN" "M20-9750242"
 			(at 59.69 86.36 0)
 			(effects
@@
 			)
 		)
-		(property "Footprint" "Connector_PinHeader_2.54mm:PinHeader_1x02_P2.54mm_Vertical"
+		(property "Footprint" "Connector_PinHeader_2.54mm:PinHeader_1x02_P2.54mm_Horizontal"
 			(at 59.69 116.84 0)
 			(effects
@@
 			)
 		)
-		(property "MPN" "61300211121"
+		(property "MPN" "M20-9750242"
 			(at 59.69 116.84 0)
 			(effects

Commit message: Releases layout for pellet, magnet, and Jetson breakout boards.
Parts:
- C32, C33, C34: LCSC (none) -> C14663; MPN CC0603ZRY5V9BB104 -> CC0603KRX7R9BB104
- J11, J15, J16, J17, J18, J21: footprint Leaf_Connectors:CONBNC002 -> Leaf_Connectors:Conn_BNC_KH-801-0038; LCSC (none) -> C2837587; MPN CONBNC002 -> KH-BNC50-3511
- J12, J13, J14: LCSC (none) -> C225269; MPN M20-9750242 -> A2005WR-2P
- R14, R15, R16, R22: LCSC (none) -> C25804; MPN RC0603FR-0710KL -> 0603WAF1002T5E
- U7: LCSC (none) -> C105266
Changed lines of the file:
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@@
 			)
 		)
-		(property "Footprint" "Leaf_Connectors:CONBNC002"
+		(property "Footprint" "Leaf_Connectors:Conn_BNC_KH-801-0038"
 			(at 48.26 34.29 0)
 			(effects
@@
 			)
 		)
-		(property "MPN" "CONBNC002"
+		(property "MPN" "KH-BNC50-3511"
+			(at 48.26 34.29 0)
+			(effects
+				(font
+					(size 1.27 1.27)
+				)
+				(hide yes)
+			)
+		)
+		(property "LCSC" "C2837587"
 			(at 48.26 34.29 0)
 			(effects
@@
 			)
 		)
-		(property "Footprint" "Leaf_Connectors:CONBNC002"
+		(property "Footprint" "Leaf_Connectors:Conn_BNC_KH-801-0038"
 			(at 49.53 153.67 0)
 			(effects
@@
 			)
 		)
-		(property "MPN" "CONBNC002"
+		(property "MPN" "KH-BNC50-3511"
+			(at 49.53 153.67 0)
+			(effects
+				(font
+					(size 1.27 1.27)
+				)
+				(hide yes)
+			)
+		)
+		(property "LCSC" "C2837587"
 			(at 49.53 153.67 0)
 			(effects
@@
 			)
 		)
-		(property "MPN" "RC0603FR-0710KL"
+		(property "MPN" "0603WAF1002T5E"
+			(at 50.8 116.84 0)
+			(effects
+				(font
+					(size 1.27 1.27)
+				)
+				(hide yes)
+			)
+		)
+		(property "LCSC" "C25804"
 			(at 50.8 116.84 0)
 			(effects
@@
 			)
 		)
-		(property "MPN" "RC0603FR-0710KL"
+		(property "MPN" "0603WAF1002T5E"
+			(at 50.8 86.36 0)
+			(effects
+				(font
+					(size 1.27 1.27)
+				)
+				(hide yes)
+			)
+		)
+		(property "LCSC" "C25804"
 			(at 50.8 86.36 0)
 			(effects
@@
 			)
 		)
-		(property "MPN" "RC0603FR-0710KL"
+		(property "MPN" "0603WAF1002T5E"
+			(at 50.8 101.6 0)
+			(effects
+				(font
+					(size 1.27 1.27)
+				)
+				(hide yes)
+			)
+		)
+		(property "LCSC" "C25804"
 			(at 50.8 101.6 0)
 			(effects
@@
 			)
 		)
-		(property "MPN" "RC0603FR-0710KL"
+		(property "MPN" "0603WAF1002T5E"
+			(at 35.56 30.48 0)
+			(effects
+				(font
+					(size 1.27 1.27)
+				)
+				(hide yes)
+			)
+		)
+		(property "LCSC" "C25804"
 			(at 35.56 30.48 0)
 			(effects
@@
 			)
 		)
-		(property "MPN" "CC0603ZRY5V9BB104"
+		(property "MPN" " CC0603KRX7R9BB104"
+			(at 39.37 38.1 0)
+			(effects
+				(font
+					(size 1.27 1.27)
+				)
+				(hide yes)
+			)
+		)
+		(property "LCSC" "C14663"
 			(at 39.37 38.1 0)
 			(effects
@@
 		)
 		(property "MPN" "TXB0104RUT"
+			(at 172.72 96.52 0)
+			(effects
+				(font
+					(size 1.27 1.27)
+				)
+				(hide yes)
+			)
+		)
+		(property "LCSC" "C105266"
 			(at 172.72 96.52 0)
 			(effects
@@
 			)
 		)
-		(property "MPN" "M20-9750242"
+		(property "MPN" " A2005WR-2P"
+			(at 59.69 101.6 0)
+			(effects
+				(font
+					(size 1.27 1.27)
+				)
+				(hide yes)
+			)
+		)
+		(property "LCSC" "C225269"
 			(at 59.69 101.6 0)
 			(effects
@@
 			)
 		)
-		(property "MPN" "M20-9750242"
+		(property "MPN" " A2005WR-2P"
+			(at 59.69 86.36 0)
+			(effects
+				(font
+					(size 1.27 1.27)
+				)
+				(hide yes)
+			)
+		)
+		(property "LCSC" "C225269"
 			(at 59.69 86.36 0)
 			(effects
@@
 			)
 		)
-		(property "Footprint" "Leaf_Connectors:CONBNC002"
+		(property "Footprint" "Leaf_Connectors:Conn_BNC_KH-801-0038"
 			(at 220.98 87.63 0)
 			(effects
@@
 			)
 		)
-		(property "MPN" "CONBNC002"
+		(property "MPN" "KH-BNC50-3511"
+			(at 220.98 87.63 0)
+			(effects
+				(font
+					(size 1.27 1.27)
+				)
+				(hide yes)
+			)
+		)
+		(property "LCSC" "C2837587"
 			(at 220.98 87.63 0)
 			(effects
@@
 			)
 		)
-		(property "Footprint" "Leaf_Connectors:CONBNC002"
+		(property "Footprint" "Leaf_Connectors:Conn_BNC_KH-801-0038"
 			(at 220.98 102.87 0)
 			(effects
@@
 			)
 		)
-		(property "MPN" "CONBNC002"
+		(property "MPN" "KH-BNC50-3511"
+			(at 220.98 102.87 0)
+			(effects
+				(font
+					(size 1.27 1.27)
+				)
+				(hide yes)
+			)
+		)
+		(property "LCSC" "C2837587"
 			(at 220.98 102.87 0)
 			(effects
@@
 			)
 		)
-		(property "MPN" "M20-9750242"
+		(property "MPN" " A2005WR-2P"
+			(at 59.69 116.84 0)
+			(effects
+				(font
+					(size 1.27 1.27)
+				)
+				(hide yes)
+			)
+		)
+		(property "LCSC" "C225269"
 			(at 59.69 116.84 0)
 			(effects
@@
 			)
 		)
-		(property "Footprint" "Leaf_Connectors:CONBNC002"
+		(property "Footprint" "Leaf_Connectors:Conn_BNC_KH-801-0038"
 			(at 220.98 71.12 0)
 			(effects
@@
 			)
 		)
-		(property "MPN" "CONBNC002"
+		(property "MPN" "KH-BNC50-3511"
+			(at 220.98 71.12 0)
+			(effects
+				(font
+					(size 1.27 1.27)
+				)
+				(hide yes)
+			)
+		)
+		(property "LCSC" "C2837587"
 			(at 220.98 71.12 0)
 			(effects
@@
 			)
 		)
-		(property "MPN" "CC0603ZRY5V9BB104"
+		(property "MPN" " CC0603KRX7R9BB104"
+			(at 179.07 76.2 0)
+			(effects
+				(font
+					(size 1.27 1.27)
+				)
+				(hide yes)
+			)
+		)
+		(property "LCSC" "C14663"
 			(at 179.07 76.2 0)
 			(effects
@@
 			)
 		)
-		(property "Footprint" "Leaf_Connectors:CONBNC002"
+		(property "Footprint" "Leaf_Connectors:Conn_BNC_KH-801-0038"
 			(at 220.98 121.92 0)
 			(effects
@@
 			)
 		)
-		(property "MPN" "CONBNC002"
+		(property "MPN" "KH-BNC50-3511"
+			(at 220.98 121.92 0)
+			(effects
+				(font
+					(size 1.27 1.27)
+				)
+				(hide yes)
+			)
+		)
+		(property "LCSC" "C2837587"
 			(at 220.98 121.92 0)
 			(effects
@@
 			)
 		)
-		(property "MPN" "CC0603ZRY5V9BB104"
+		(property "MPN" " CC0603KRX7R9BB104"
 			(at 166.37 76.2 0)
 			(effects
+				(font
+					(size 1.27 1.27)
+				)
+				(hide yes)
+			)
+		)
+		(property "LCSC" "C14663"
+			(at 166.37 76.2 0)
+			(effects
