File: hardware/pellet_module/power.kicad_sch (KiCad schematic)
At the start: 29 parts, among them J22 Barrel_Jack_Switch, U8 TPS561201, U9 TPS565208

Commit message: Fixes based on discovered issues on testing rig
Other:
- note added: "Expected current consumption: 126mA"
- note removed: "Expected current consumption: 126mA Supports max 500mA"
Changed lines of the file:
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@@
 		)
 	)
-	(text "Expected current consumption: 126mA\nSupports max 500mA"
+	(text "Expected current consumption: 126mA"
 		(exclude_from_sim no)
 		(at 139.954 138.684 0)

Commit message: Update Pellet BOM for part availability
Parts:
- R20: LCSC C185321 -> C23077
Changed lines of the file:
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@@
 			)
 		)
-		(property "LCSC" "C185321"
+		(property "LCSC" "C23077"
 			(at 205.74 78.74 0)
 			(effects
